Commit message: working ideantification, no fitting yet

File: src/robots/urdf/test_robot.urdf (robot description, URDF)
Before this commit: robot sbot, 12 links, 11 joints
Links:
- removed link base
- removed link flange
- removed link scene_environment
- removed link tool0
- removed link world
Joints:
- removed joint base_joint
- removed joint base_link-base_joint
- removed joint base_to_scene
- removed joint joint5-tool0
- removed joint tool0-flange_joint
